Commit message: finish orientation calculation

File: nbv_code/ros2_ws2/install/my_bot/share/my_bot/description/gazebo_control.xacro (robot description, xacro)
@@ -14,5 +14,5 @@
             <!-- output 告訴說這個plugin要output什麼-->
             <odometry_frame>odom</odometry_frame>
-            <robot_base_frame>base_link</robot_base_frame>
+            <robot_base_frame>base</robot_base_frame>
             <publish_odom>true</publish_odom>
             <publish_odom_tf>true</publish_odom_tf>

File: nbv_code/ros2_ws2/install/my_bot/share/my_bot/description/robot_core.xacro (robot description, xacro)
@@ -31,9 +31,9 @@
     -->
     <!-- set baselink(1st link for mobile robot) -->
-    <link name="base_link">
+    <link name="base">
     </link>
     <!-- box link -->
     <joint name="chassis_joint" type="fixed">
-        <parent link="base_link"/>
+        <parent link="base"/>
         <child link="chassis"/>
         <origin xyz="-0.1 0 0"/> <!-- car_box link"的origin" 和base link的相對位置-->
@@ -68,5 +68,5 @@
     <!-- Left wheel link -->
     <joint name="left_wheel_joint" type="continuous"><!-- 因為車車輪子會contunuously轉 -->
-        <parent link="base_link"/>
+        <parent link="base"/>
         <child link="left_wheel"/>
         <origin xyz="0.0 0.175 0.0" rpy="-${pi/2} 0 0"/><!-- 因為在ros defult 的cylindeer是直統向上的,但輪子我們想讓它以x為軸去轉90度轉向側邊（想要輪子的z指向世界的外邊) -->
@@ -95,5 +95,5 @@
     <!-- Right wheel link -->
     <joint name="right_wheel_joint" type="continuous"><!-- 因為車車輪子會contunuously轉 -->
-        <parent link="base_link"/>
+        <parent link="base"/>
         <child link="right_wheel"/><!--origin xyz: 相對於parrent link的相對座標-->
         <origin xyz="0.0 -0.175 0.0" rpy="+${pi/2} 0 0"/><!-- 因為在ros defult 的cylindeer是直統向上的,但輪子我們想讓它以x為軸去轉90度轉向側邊（想要輪子的z指向世界的外邊) -->
